File: designer/public/templates/BeagleBone-Black-Cape/BeagleBone-Black-Cape.kicad_pcb (KiCad board)
At the start: 2 copper layers, 86.4 x 54.6 mm, 6 parts, among them P8 BeagleBone_Black_Header, P9 BeagleBone_Black_Header

Commit message: designer: make the project manager indistinguishable from KiCad's
An engineer arriving from KiCad should not be able to tell the two windows
apart. This is that pass over the manager frame, ported from the 10.0.5 source
the user runs rather than from screenshots, with the screenshots used only to
settle the colours GTK paints rather than KiCad.

The palette drops the blue tint it had for the neutral greys the theme
actually uses, and the shell adopts wxSYS_DEFAULT_GUI_FONT's 11pt in the menu
bar, tree, launcher, status bar, buttons and dialog headers.

PANEL_KICAD_LAUNCHER: the tile order and tooltips come from CreateLaunchers(),
the New Project icon is new_project_from_template as KICAD_MANAGER_ACTIONS
names it, and the hover box is the 56px button - a 48px bitmap plus
SetPadding(4) - not the 760px row, so hovering the label no longer lights it.
BITMAP_BUTTON::OnPaint draws a rectangle, hence the square corners. The Plugin
and Content Manager tile and its menu entry are gone for now.

PROJECT_TREE_PANE: selection hugs the icon and label rather than the row,
because wxTR_FULL_ROW_HIGHLIGHT appears nowhere in KiCad; single click
selects and only double click expands; and the file list is
s_allowedExtensionsToList transcribed, an allow list with no .step or .wrl -
which is why a .3dshapes folder gets no expander. The pane width persists as
m_LeftWinWidth does.

KISTATUSBAR ellipsizes the middle of the project path the way
SetEllipsedTextField does, minus the width of "XX"; ellipsize.ts is that
wxELLIPSIZE_MIDDLE port.

DIALOG_TEMPLATE_SELECTOR is rebuilt against 10.0.5, which differs from master
here: three filter choices rather than four, no Browse/Clear row, and cards
labelled with the template's directory name, because PROJECT_TEMPLATE's
constructor assigns m_title = GetPrjDirName() and leaves GetTitle()'s HTML
parse unreachable. tools/templates/import.mjs derives title, description and
file list the same three ways the C++ does and imports all 20 templates with
th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
Connections:
- P8 pad 35: /LCD.DATA8 -> /LCD.DATA12
- P8 pad 37: /LCD.DATA6 -> /LCD.DATA8
- P8 pad 39: /LCD.DATA4 -> /LCD.DATA6
- P8 pad 41: /LCD.DATA2 -> /LCD.DATA4
- P8 pad 43: /LCD.DATA0 -> /LCD.DATA2
- P8 pad 45: GNDD -> /LCD.DATA0
